File: hardware/design/Main Board/Sheet 2.sch (KiCad schematic (older format))
At the start: 24 parts

Commit message: Version 1.0.051414.2106
- Added JTAG & Programming Port to MCU.
- Moved I2C Display to the I2C2 Buss.
- Added 10K reference resistors.
Parts:
- removed C? (x4): 100n, ~, symbol C
- added R? (x4): 10K, ~, symbol R
Connections:
- wire segments 67 -> 59
Other:
- note added: "All Resistors 0.1%\n"
Changed lines of the file:
@@
 Sheet 2 9
 Title "Hybrid Audio Dynamics Processor"
-Date "11 may 2014"
+Date "15 may 2014"
 Rev "1.0"
 Comp "P14345"
@@
 $EndComp
 $Comp
-L C C?
-U 1 1 534DBD6E
-P 4875 2250
-F 0 "C?" V 4925 2350 40  0000 L CNN
-F 1 "100n" V 4925 2050 40  0000 L CNN
-F 2 "~" H 4913 2100 30  0000 C CNN
-F 3 "~" H 4875 2250 60  0000 C CNN
-	1    4875 2250
-	0    -1   -1   0
-$EndComp
-$Comp
-L C C?
-U 1 1 534DBD7D
-P 4875 3250
-F 0 "C?" V 4925 3375 40  0000 L CNN
-F 1 "100n" V 4925 3050 40  0000 L CNN
-F 2 "~" H 4913 3100 30  0000 C CNN
-F 3 "~" H 4875 3250 60  0000 C CNN
-	1    4875 3250
-	0    -1   -1   0
-$EndComp
-$Comp
 L R R?
 U 1 1 534DBD8A
@@
 $EndComp
 $Comp
-L C C?
-U 1 1 534DBDE2
-P 4925 4650
-F 0 "C?" V 4975 4725 40  0000 L CNN
-F 1 "100n" V 4975 4450 40  0000 L CNN
-F 2 "~" H 4963 4500 30  0000 C CNN
-F 3 "~" H 4925 4650 60  0000 C CNN
-	1    4925 4650
-	0    -1   -1   0
-$EndComp
-$Comp
-L C C?
-U 1 1 534DBDE8
-P 4925 5650
-F 0 "C?" V 4975 5725 40  0000 L CNN
-F 1 "100n" V 4975 5450 40  0000 L CNN
-F 2 "~" H 4963 5500 30  0000 C CNN
-F 3 "~" H 4925 5650 60  0000 C CNN
-	1    4925 5650
-	0    -1   -1   0
-$EndComp
-$Comp
 L R R?
 U 1 1 534DBDEE
@@
 	5075 2600 5275 2600
 Wire Wire Line
-	5075 2250 5175 2250
-Wire Wire Line
-	5175 2250 5175 2600
-Connection ~ 5175 2600
-Wire Wire Line
 	5075 2950 5275 2950
-Wire Wire Line
-	5075 3250 5175 3250
-Wire Wire Line
-	5175 3250 5175 2950
-Connection ~ 5175 2950
 Wire Wire Line
 	5775 2600 6075 2600
@@
 	4675 2950 4325 2950
 Wire Wire Line
-	4675 3250 4575 3250
-Wire Wire Line
-	4575 3250 4575 2950
-Connection ~ 4575 2950
-Wire Wire Line
 	4675 2600 4325 2600
 Wire Wire Line
-	4675 2250 4575 2250
-Wire Wire Line
-	4575 2250 4575 2600
-Connection ~ 4575 2600
-Wire Wire Line
 	5125 5000 5325 5000
 Wire Wire Line
 	5125 5350 5325 5350
 Wire Wire Line
-	5125 4650 5225 4650
-Wire Wire Line
-	5225 4650 5225 5000
-Connection ~ 5225 5000
-Wire Wire Line
-	5125 5650 5225 5650
-Wire Wire Line
-	5225 5650 5225 5350
-Connection ~ 5225 5350
-Wire Wire Line
 	4325 5000 4725 5000
 Wire Wire Line
-	4725 4650 4625 4650
-Wire Wire Line
-	4625 4650 4625 5000
-Connection ~ 4625 5000
-Wire Wire Line
 	4725 5350 4325 5350
-Wire Wire Line
-	4725 5650 4625 5650
-Wire Wire Line
-	4625 5650 4625 5350
-Connection ~ 4625 5350
 Wire Wire Line
 	5825 5350 6125 5350
@@
 Connection ~ 6775 2450
 Connection ~ 6775 3100
+Text Notes 5350 6600 0    100  ~ 0
+All Resistors 0.1%\n
+$Comp
+L R R?
+U 1 1 5374A1ED
+P 4550 3300
+F 0 "R?" V 4630 3300 40  0000 C CNN
+F 1 "10K" V 4557 3301 40  0000 C CNN
+F 2 "~" V 4480 3300 30  0000 C CNN
+F 3 "~" H 4550 3300 30  0000 C CNN
+	1    4550 3300
+	1    0    0    -1
+$EndComp
+$Comp
+L R R?
+U 1 1 5374A201
+P 4550 2250
+F 0 "R?" V 4630 2250 40  0000 C CNN
+F 1 "10K" V 4557 2251 40  0000 C CNN
+F 2 "~" V 4480 2250 30  0000 C CNN
+F 3 "~" H 4550 2250 30  0000 C CNN
+	1    4550 2250
+	1    0    0    -1
+$EndComp
+$Comp
+L R R?
+U 1 1 5374A207
+P 4550 4650
+F 0 "R?" V 4630 4650 40  0000 C CNN
+F 1 "10K" V 4557 4651 40  0000 C CNN
+F 2 "~" V 4480 4650 30  0000 C CNN
+F 3 "~" H 4550 4650 30  0000 C CNN
+	1    4550 4650
+	1    0    0    -1
+$EndComp
+$Comp
+L R R?
+U 1 1 5374A20D
+P 4550 5700
+F 0 "R?" V 4630 5700 40  0000 C CNN
+F 1 "10K" V 4557 5701 40  0000 C CNN
+F 2 "~" V 4480 5700 30  0000 C CNN
+F 3 "~" H 4550 5700 30  0000 C CNN
+	1    4550 5700
+	1    0    0    -1
+$EndComp
+Wire Wire Line
+	4550 2500 4550 2600
+Connection ~ 4550 2600
+Wire Wire Line
+	4550 3050 4550 2950
+Connection ~ 4550 2950
+Wire Wire Line
+	4550 4900 4550 5000
+Connection ~ 4550 5000
+Wire Wire Line
+	4550 5450 4550 5350
+Connection ~ 4550 5350
+Wire Wire Line
+	4550 5950 4550 6000
+Wire Wire Line
+	4550 4400 4550 4350
+Wire Wire Line
+	4550 3550 4550 3600
+Wire Wire Line
+	4550 2000 4550 1950
+$Comp
+L GND #PWR?
+U 1 1 5374A46B
+P 4550 1950
+F 0 "#PWR?" H 4550 1950 30  0001 C CNN
+F 1 "GND" H 4550 1880 30  0001 C CNN
+F 2 "" H 4550 1950 60  0000 C CNN
+F 3 "" H 4550 1950 60  0000 C CNN
+	1    4550 1950
+	-1   0    0    1
+$EndComp
+$Comp
+L GND #PWR?
+U 1 1 5374A47A
+P 4550 3600
+F 0 "#PWR?" H 4550 3600 30  0001 C CNN
+F 1 "GND" H 4550 3530 30  0001 C CNN
+F 2 "" H 4550 3600 60  0000 C CNN
+F 3 "" H 4550 3600 60  0000 C CNN
+	1    4550 3600
+	1    0    0    -1
+$EndComp
+$Comp
+L GND #PWR?
+U 1 1 5374A489
+P 4550 4350
+F 0 "#PWR?" H 4550 4350 30  0001 C CNN
+F 1 "GND" H 4550 4280 30  0001 C CNN
+F 2 "" H 4550 4350 60  0000 C CNN
+F 3 "" H 4550 4350 60  0000 C CNN
+	1    4550 4350
+	-1   0    0    1
+$EndComp
+$Comp
+L GND #PWR?
+U 1 1 5374A498
+P 4550 6000
+F 0 "#PWR?" H 4550 6000 30  0001 C CNN
+F 1 "GND" H 4550 5930 30  0001 C CNN
+F 2 "" H 4550 6000 60  0000 C CNN
+F 3 "" H 4550 6000 60  0000 C CNN
+	1    4550 6000
+	1    0    0    -1
+$EndComp
 $EndSCHEMATC

Commit message: Version 1.0.082514.2134
Initial partial PCB layout.
Parts:
- added P3, P4, P5, P6, P7, P8: TST, ~, symbol TST
- gave numbers to parts that had none: 23
Connections:
- wire segments 59 -> 65
Changed lines of the file:
@@
 Sheet 2 9
 Title "Hybrid Audio Dynamics Processor"
-Date "15 may 2014"
+Date "26 aug 2014"
 Rev "1.0"
 Comp "P14345"
@@
 $EndDescr
 $Comp
-L OPA2134 U?
+L OPA2134 U1
 U 1 1 534DBCB9
 P 6825 2750
-F 0 "U?" H 6950 2475 60  0000 L CNN
+F 0 "U1" H 6950 2475 60  0000 L CNN
 F 1 "OP275" H 6925 2550 60  0000 L CNN
 F 2 "" H 6825 2750 60  0000 C CNN
@@
 $EndComp
 $Comp
-L OPA2134 U?
+L OPA2134 U1
 U 2 1 534DBCE6
 P 6875 5150
-F 0 "U?" H 6875 5450 60  0000 L CNN
+F 0 "U1" H 6875 5450 60  0000 L CNN
 F 1 "OP275" H 6850 5350 60  0000 L CNN
 F 2 "" H 6875 5150 60  0000 C CNN
@@
 $EndComp
 $Comp
-L CP1 C?
+L CP1 C1
 U 1 1 534DBD13
 P 4875 2600
-F 0 "C?" V 4925 2700 50  0000 L CNN
+F 0 "C1" V 4925 2700 50  0000 L CNN
 F 1 "22u" V 4925 2400 50  0000 L CNN
 F 2 "~" H 4875 2600 60  0000 C CNN
@@
 $EndComp
 $Comp
-L CP1 C?
+L CP1 C2
 U 1 1 534DBD22
 P 4875 2950
-F 0 "C?" V 4925 3050 50  0000 L CNN
+F 0 "C2" V 4925 3050 50  0000 L CNN
 F 1 "22u" V 4925 2750 50  0000 L CNN
 F 2 "~" H 4875 2950 60  0000 C CNN
@@
 $EndComp
 $Comp
-L R R?
+L R R5
 U 1 1 534DBD31
 P 5525 2600
-F 0 "R?" V 5605 2600 40  0000 C CNN
+F 0 "R5" V 5605 2600 40  0000 C CNN
 F 1 "22K" V 5532 2601 40  0000 C CNN
 F 2 "~" V 5455 2600 30  0000 C CNN
@@
 $EndComp
 $Comp
-L R R?
+L R R6
 U 1 1 534DBD5C
 P 5525 2950
-F 0 "R?" V 5605 2950 40  0000 C CNN
+F 0 "R6" V 5605 2950 40  0000 C CNN
 F 1 "22K" V 5532 2951 40  0000 C CNN
 F 2 "~" V 5455 2950 30  0000 C CNN
@@
 $EndComp
 $Comp
-L R R?
+L R R9
 U 1 1 534DBD8A
 P 6175 3200
-F 0 "R?" V 6255 3200 40  0000 C CNN
+F 0 "R9" V 6255 3200 40  0000 C CNN
 F 1 "22K" V 6182 3201 40  0000 C CNN
 F 2 "~" V 6105 3200 30  0000 C CNN
@@
 $EndComp
 $Comp
-L C C?
+L C C5
 U 1 1 534DBDA4
 P 6425 3200
-F 0 "C?" H 6425 3300 40  0000 L CNN
+F 0 "C5" H 6425 3300 40  0000 L CNN
 F 1 "33p" H 6431 3115 40  0000 L CNN
 F 2 "~" H 6463 3050 30  0000 C CNN
@@
 $EndComp
 $Comp
-L R R?
+L R R11
 U 1 1 534DBDAA
 P 6625 2200
-F 0 "R?" V 6705 2200 40  0000 C CNN
+F 0 "R11" V 6705 2200 40  0000 C CNN
 F 1 "22K" V 6632 2201 40  0000 C CNN
 F 2 "~" V 6555 2200 30  0000 C CNN
@@
 $EndComp
 $Comp
-L C C?
+L C C7
 U 1 1 534DBDB0
 P 6625 1950
-F 0 "C?" V 6675 2025 40  0000 L CNN
+F 0 "C7" V 6675 2025 40  0000 L CNN
 F 1 "33p" V 6675 1775 40  0000 L CNN
 F 2 "~" H 6663 1800 30  0000 C CNN
@@
 $EndComp
 $Comp
-L CP1 C?
+L CP1 C3
 U 1 1 534DBDCA
 P 4925 5000
-F 0 "C?" V 4975 5100 50  0000 L CNN
+F 0 "C3" V 4975 5100 50  0000 L CNN
 F 1 "22u" V 4975 4800 50  0000 L CNN
 F 2 "~" H 4925 5000 60  0000 C CNN
@@
 $EndComp
 $Comp
-L CP1 C?
+L CP1 C4
 U 1 1 534DBDD0
 P 4925 5350
-F 0 "C?" V 4975 5450 50  0000 L CNN
+F 0 "C4" V 4975 5450 50  0000 L CNN
 F 1 "22u" V 4975 5150 50  0000 L CNN
 F 2 "~" H 4925 5350 60  0000 C CNN
@@
 $EndComp
 $Comp
-L R R?
+L R R7
 U 1 1 534DBDD6
 P 5575 5000
-F 0 "R?" V 5655 5000 40  0000 C CNN
+F 0 "R7" V 5655 5000 40  0000 C CNN
 F 1 "22K" V 5582 5001 40  0000 C CNN
 F 2 "~" V 5505 5000 30  0000 C CNN
@@
 $EndComp
 $Comp
-L R R?
+L R R8
 U 1 1 534DBDDC
 P 5575 5350
-F 0 "R?" V 5655 5350 40  0000 C CNN
+F 0 "R8" V 5655 5350 40  0000 C CNN
 F 1 "22K" V 5582 5351 40  0000 C CNN
 F 2 "~" V 5505 5350 30  0000 C CNN
@@
 $EndComp
 $Comp
-L R R?
+L R R10
 U 1 1 534DBDEE
 P 6225 5600
-F 0 "R?" V 6305 5600 40  0000 C CNN
+F 0 "R10" V 6305 5600 40  0000 C CNN
 F 1 "22K" V 6232 5601 40  0000 C CNN
 F 2 "~" V 6155 5600 30  0000 C CNN
@@
 $EndComp
 $Comp
-L C C?
+L C C6
 U 1 1 534DBDF4
 P 6475 5600
-F 0 "C?" H 6475 5700 40  0000 L CNN
+F 0 "C6" H 6475 5700 40  0000 L CNN
 F 1 "33p" H 6481 5515 40  0000 L CNN
 F 2 "~" H 6513 5450 30  0000 C CNN
@@
 $EndComp
 $Comp
-L R R?
+L R R12
 U 1 1 534DBDFA
 P 6675 4600
-F 0 "R?" V 6755 4600 40  0000 C CNN
+F 0 "R12" V 6755 4600 40  0000 C CNN
 F 1 "22K" V 6682 4601 40  0000 C CNN
 F 2 "~" V 6605 4600 30  0000 C CNN
@@
 $EndComp
 $Comp
-L C C?
+L C C8
 U 1 1 534DBE00
 P 6675 4350
-F 0 "C?" V 6725 4425 40  0000 L CNN
+F 0 "C8" V 6725 4425 40  0000 L CNN
 F 1 "33p" V 6725 4150 40  0000 L CNN
 F 2 "~" H 6713 4200 30  0000 C CNN
@@
 	6475 6000 6475 5800
 $Comp
-L CSMALL C?
+L CSMALL C9
 U 1 1 534DC611
 P 6875 2450
-F 0 "C?" V 6925 2475 30  0000 L CNN
+F 0 "C9" V 6925 2475 30  0000 L CNN
 F 1 "0.1u" V 6925 2325 30  0000 L CNN
 F 2 "~" H 6875 2450 60  0000 C CNN
@@
 $EndComp
 $Comp
-L CSMALL C?
+L CSMALL C10
 U 1 1 534DC620
 P 6875 3100
-F 0 "C?" V 6925 3025 30  0000 L CNN
+F 0 "C10" V 6925 3025 30  0000 L CNN
 F 1 "0.1u" V 6925 3125 30  0000 L CNN
 F 2 "~" H 6875 3100 60  0000 C CNN
@@
 $EndComp
 $Comp
-L GND #PWR?
+L GND #PWR01
 U 1 1 534DC69D
 P 6300 3675
-F 0 "#PWR?" H 6300 3675 30  0001 C CNN
+F 0 "#PWR01" H 6300 3675 30  0001 C CNN
 F 1 "GND" H 6300 3605 30  0001 C CNN
 F 2 "" H 6300 3675 60  0000 C CNN
@@
 $EndComp
 $Comp
-L GND #PWR?
+L GND #PWR02
 U 1 1 534DC6AC
 P 6350 6075
-F 0 "#PWR?" H 6350 6075 30  0001 C CNN
+F 0 "#PWR02" H 6350 6075 30  0001 C CNN
 F 1 "GND" H 6350 6005 30  0001 C CNN
 F 2 "" H 6350 6075 60  0000 C CNN
@@
 $EndComp
 $Comp
-L GND #PWR?
+L GND #PWR03
 U 1 1 534DC6BB
 P 7025 3200
-F 0 "#PWR?" H 7025 3200 30  0001 C CNN
+F 0 "#PWR03" H 7025 3200 30  0001 C CNN
 F 1 "GND" H 7025 3130 30  0001 C CNN
 F 2 "" H 7025 3200 60  0000 C CNN
@@
 $EndComp
 $Comp
-L GND #PWR?
+L GND #PWR04
 U 1 1 534DC6CA
 P 7025 2525
-F 0 "#PWR?" H 7025 2525 30  0001 C CNN
+F 0 "#PWR04" H 7025 2525 30  0001 C CNN
 F 1 "GND" H 7025 2455 30  0001 C CNN
 F 2 "" H 7025 2525 60  0000 C CNN
@@
 CH2
 $Comp
-L VSS #PWR?
+L VSS #PWR05
 U 1 1 535FAFA8
 P 6775 3225
-F 0 "#PWR?" H 6775 3225 30  0001 C CNN
+F 0 "#PWR05" H 6775 3225 30  0001 C CNN
 F 1 "VSS" H 6775 3155 30  0000 C CNN
 F 2 "" H 6775 3225 60  0000 C CNN
@@
 $EndComp
 $Comp
-L VDD #PWR?
+L VDD #PWR06
 U 1 1 535FAFDA
 P 6775 2425
-F 0 "#PWR?" H 6775 2525 30  0001 C CNN
+F 0 "#PWR06" H 6775 2525 30  0001 C CNN
 F 1 "VDD" H 6775 2535 30  0000 C CNN
 F 2 "" H 6775 2425 60  0000 C CNN
@@
 All Resistors 0.1%\n
 $Comp
-L R R?
+L R R2
 U 1 1 5374A1ED
 P 4550 3300
-F 0 "R?" V 4630 3300 40  0000 C CNN
+F 0 "R2" V 4630 3300 40  0000 C CNN
 F 1 "10K" V 4557 3301 40  0000 C CNN
 F 2 "~" V 4480 3300 30  0000 C CNN
@@
 $EndComp
 $Comp
-L R R?
+L R R1
 U 1 1 5374A201
 P 4550 2250
-F 0 "R?" V 4630 2250 40  0000 C CNN
+F 0 "R1" V 4630 2250 40  0000 C CNN
 F 1 "10K" V 4557 2251 40  0000 C CNN
 F 2 "~" V 4480 2250 30  0000 C CNN
@@
 $EndComp
 $Comp
-L R R?
+L R R3
 U 1 1 5374A207
 P 4550 4650
-F 0 "R?" V 4630 4650 40  0000 C CNN
+F 0 "R3" V 4630 4650 40  0000 C CNN
 F 1 "10K" V 4557 4651 40  0000 C CNN
 F 2 "~" V 4480 4650 30  0000 C CNN
@@
 $EndComp
 $Comp
-L R R?
+L R R4
 U 1 1 5374A20D
 P 4550 5700
-F 0 "R?" V 4630 5700 40  0000 C CNN
+F 0 "R4" V 4630 5700 40  0000 C CNN
 F 1 "10K" V 4557 5701 40  0000 C CNN
 F 2 "~" V 4480 5700 30  0000 C CNN
@@
 	4550 2000 4550 1950
 $Comp
-L GND #PWR?
+L GND #PWR07
 U 1 1 5374A46B
 P 4550 1950
-F 0 "#PWR?" H 4550 1950 30  0001 C CNN
+F 0 "#PWR07" H 4550 1950 30  0001 C CNN
 F 1 "GND" H 4550 1880 30  0001 C CNN
 F 2 "" H 4550 1950 60  0000 C CNN
@@
 $EndComp
 $Comp
-L GND #PWR?
+L GND #PWR08
 U 1 1 5374A47A
 P 4550 3600
-F 0 "#PWR?" H 4550 3600 30  0001 C CNN
+F 0 "#PWR08" H 4550 3600 30  0001 C CNN
 F 1 "GND" H 4550 3530 30  0001 C CNN
 F 2 "" H 4550 3600 60  0000 C CNN
@@
 $EndComp
 $Comp
-L GND #PWR?
+L GND #PWR09
 U 1 1 5374A489
 P 4550 4350
-F 0 "#PWR?" H 4550 4350 30  0001 C CNN
+F 0 "#PWR09" H 4550 4350 30  0001 C CNN
 F 1 "GND" H 4550 4280 30  0001 C CNN
 F 2 "" H 4550 4350 60  0000 C CNN
@@
 $EndComp
 $Comp
-L GND #PWR?
+L GND #PWR010
 U 1 1 5374A498
 P 4550 6000
-F 0 "#PWR?" H 4550 6000 30  0001 C CNN
+F 0 "#PWR010" H 4550 6000 30  0001 C CNN
 F 1 "GND" H 4550 5930 30  0001 C CNN
 F 2 "" H 4550 6000 60  0000 C CNN
@@
 	1    0    0    -1
 $EndComp
+$Comp
+L TST P3
+U 1 1 53DE6438
+P 4400 2550
+F 0 "P3" H 4400 2850 40  0000 C CNN
+F 1 "TST" H 4400 2800 30  0000 C CNN
+F 2 "~" H 4400 2550 60  0000 C CNN
+F 3 "~" H 4400 2550 60  0000 C CNN
+	1    4400 2550
+	1    0    0    -1
+$EndComp
+$Comp
+L TST P4
+U 1 1 53DE6447
+P 4400 3000
+F 0 "P4" H 4400 3300 40  0000 C CNN
+F 1 "TST" H 4400 3250 30  0000 C CNN
+F 2 "~" H 4400 3000 60  0000 C CNN
+F 3 "~" H 4400 3000 60  0000 C CNN
+	1    4400 3000
+	-1   0    0    1
+$EndComp
+$Comp
+L TST P7
+U 1 1 53DE6456
+P 7350 1900
+F 0 "P7" H 7350 2200 40  0000 C CNN
+F 1 "TST" H 7350 2150 30  0000 C CNN
+F 2 "~" H 7350 1900 60  0000 C CNN
+F 3 "~" H 7350 1900 60  0000 C CNN
+	1    7350 1900
+	1    0    0    -1
+$EndComp
+$Comp
+L TST P5
+U 1 1 53DE6465
+P 4400 4950
+F 0 "P5" H 4400 5250 40  0000 C CNN
+F 1 "TST" H 4400 5200 30  0000 C CNN
+F 2 "~" H 4400 4950 60  0000 C CNN
+F 3 "~" H 4400 4950 60  0000 C CNN
+	1    4400 4950
+	1    0    0    -1
+$EndComp
+$Comp
+L TST P6
+U 1 1 53DE6474
+P 4400 5400
+F 0 "P6" H 4400 5700 40  0000 C CNN
+F 1 "TST" H 4400 5650 30  0000 C CNN
+F 2 "~" H 4400 5400 60  0000 C CNN
+F 3 "~" H 4400 5400 60  0000 C CNN
+	1    4400 5400
+	-1   0    0    1
+$EndComp
+$Comp
+L TST P8
+U 1 1 53DE6483
+P 7350 4300
+F 0 "P8" H 7350 4600 40  0000 C CNN
+F 1 "TST" H 7350 4550 30  0000 C CNN
+F 2 "~" H 7350 4300 60  0000 C CNN
+F 3 "~" H 7350 4300 60  0000 C CNN
+	1    7350 4300
+	1    0    0    -1
+$EndComp
+Wire Wire Line
+	4400 3000 4400 2950
+Connection ~ 4400 2950
+Wire Wire Line
+	4400 2550 4400 2600
+Connection ~ 4400 2600
+Wire Wire Line
+	4400 4950 4400 5000
+Connection ~ 4400 5000
+Wire Wire Line
+	4400 5400 4400 5350
+Connection ~ 4400 5350
+Wire Wire Line
+	7350 1900 7350 1950
+Connection ~ 7350 1950
+Wire Wire Line
+	7350 4300 7350 4350
+Connection ~ 7350 4350
 $EndSCHEMATC

Commit message: Version 1.0.090114.2238
Completed Layout
Parts:
- added R100, R101: 0, ~, symbol R
Connections:
- wire segments 65 -> 67
Changed lines of the file:
@@
 Sheet 2 9
 Title "Hybrid Audio Dynamics Processor"
-Date "26 aug 2014"
+Date "2 sep 2014"
 Rev "1.0"
 Comp "P14345"
@@
 Connection ~ 7375 2750
 Connection ~ 7375 5150
-Text HLabel 7500 2750 2    60   Output ~ 0
+Text HLabel 8100 2750 2    60   Output ~ 0
 CH1
-Text HLabel 7500 5150 2    60   Output ~ 0
+Text HLabel 8100 5150 2    60   Output ~ 0
 CH2
 $Comp
@@
 	7350 4300 7350 4350
 Connection ~ 7350 4350
+$Comp
+L R R100
+U 1 1 54051DA8
+P 7750 2750
+F 0 "R100" V 7830 2750 40  0000 C CNN
+F 1 "0" V 7757 2751 40  0000 C CNN
+F 2 "~" V 7680 2750 30  0000 C CNN
+F 3 "~" H 7750 2750 30  0000 C CNN
+	1    7750 2750
+	0    -1   -1   0
+$EndComp
+$Comp
+L R R101
+U 1 1 54051DB7
+P 7750 5150
+F 0 "R101" V 7830 5150 40  0000 C CNN
+F 1 "0" V 7757 5151 40  0000 C CNN
+F 2 "~" V 7680 5150 30  0000 C CNN
+F 3 "~" H 7750 5150 30  0000 C CNN
+	1    7750 5150
+	0    -1   -1   0
+$EndComp
+Wire Wire Line
+	8000 2750 8100 2750
+Wire Wire Line
+	8000 5150 8100 5150
 $EndSCHEMATC
