File: hardware/design/Main Board/Sheet 3.sch (KiCad schematic (older format))
At the start: 22 parts

Commit message: Added Power Ports
Parts:
- removed U?: NE5532, symbol NE5532
- added U?: NE5532, ~, symbol NE5532
Connections:
- net labels added: VDD, VSS
Changed lines of the file:
@@
 Sheet 3 5
 Title ""
-Date "17 apr 2014"
+Date "29 apr 2014"
 Rev ""
 Comp ""
@@
 $EndComp
 $Comp
-L NE5532 U?
-U 1 1 534DD258
-P 6900 5050
-F 0 "U?" H 6900 5350 60  0000 L CNN
-F 1 "NE5532" H 6900 5250 60  0000 L CNN
-F 2 "" H 6900 5050 60  0000 C CNN
-F 3 "" H 6900 5050 60  0000 C CNN
-	1    6900 5050
-	1    0    0    1
-$EndComp
-$Comp
 L R R?
 U 1 1 534DD25E
@@
 $EndComp
 Wire Wire Line
-	4750 2500 4750 2550
-Wire Wire Line
-	4750 3050 4750 3100
-Wire Wire Line
-	4750 4700 4750 4650
-Wire Wire Line
-	4750 5200 4750 5250
+	4750 2450 4750 2550
+Wire Wire Line
+	4750 3050 4750 3200
+Wire Wire Line
+	4750 4600 4750 4700
+Wire Wire Line
+	4750 5200 4750 5350
 $Comp
 L GND #PWR?
@@
 Text HLabel 7800 5050 2    60   Output ~ 0
 CH2_RECT_OUT
+$Comp
+L VDD #PWR?
+U 1 1 535FB36E
+P 4750 2450
+F 0 "#PWR?" H 4750 2550 30  0001 C CNN
+F 1 "VDD" H 4750 2560 30  0000 C CNN
+F 2 "" H 4750 2450 60  0000 C CNN
+F 3 "" H 4750 2450 60  0000 C CNN
+	1    4750 2450
+	1    0    0    -1
+$EndComp
+$Comp
+L VSS #PWR?
+U 1 1 535FB37D
+P 4750 3200
+F 0 "#PWR?" H 4750 3200 30  0001 C CNN
+F 1 "VSS" H 4750 3130 30  0000 C CNN
+F 2 "" H 4750 3200 60  0000 C CNN
+F 3 "" H 4750 3200 60  0000 C CNN
+	1    4750 3200
+	1    0    0    -1
+$EndComp
+Connection ~ 4750 2500
+Connection ~ 4750 3100
+$Comp
+L VSS #PWR?
+U 1 1 535FB427
+P 4750 5350
+F 0 "#PWR?" H 4750 5350 30  0001 C CNN
+F 1 "VSS" H 4750 5280 30  0000 C CNN
+F 2 "" H 4750 5350 60  0000 C CNN
+F 3 "" H 4750 5350 60  0000 C CNN
+	1    4750 5350
+	1    0    0    -1
+$EndComp
+$Comp
+L VDD #PWR?
+U 1 1 535FB436
+P 4750 4600
+F 0 "#PWR?" H 4750 4700 30  0001 C CNN
+F 1 "VDD" H 4750 4710 30  0000 C CNN
+F 2 "" H 4750 4600 60  0000 C CNN
+F 3 "" H 4750 4600 60  0000 C CNN
+	1    4750 4600
+	1    0    0    -1
+$EndComp
+Connection ~ 4750 4650
+Connection ~ 4750 5250
+$Comp
+L NE5532 U?
+U 2 1 535FB5D4
+P 6900 5050
+F 0 "U?" H 6900 5350 60  0000 L CNN
+F 1 "NE5532" H 6900 5250 60  0000 L CNN
+F 2 "~" H 6900 5050 60  0000 C CNN
+F 3 "~" H 6900 5050 60  0000 C CNN
+	2    6900 5050
+	1    0    0    -1
+$EndComp
 $EndSCHEMATC

Commit message: Op Amp Changes
Parts:
- U? (x4): value NE5532 -> OP275
Changed lines of the file:
@@
 $Descr A4 11693 8268
 encoding utf-8
-Sheet 3 5
+Sheet 3 6
 Title ""
-Date "29 apr 2014"
+Date "2 may 2014"
 Rev ""
 Comp ""
@@
 P 4800 2800
 F 0 "U?" H 5000 2700 60  0000 L CNN
-F 1 "NE5532" H 4975 2625 60  0000 L CNN
+F 1 "OP275" H 4975 2625 60  0000 L CNN
 F 2 "" H 4800 2800 60  0000 C CNN
 F 3 "" H 4800 2800 60  0000 C CNN
@@
 P 6900 2900
 F 0 "U?" H 6900 3200 60  0000 L CNN
-F 1 "NE5532" H 6900 3100 60  0000 L CNN
+F 1 "OP275" H 6900 3100 60  0000 L CNN
 F 2 "" H 6900 2900 60  0000 C CNN
 F 3 "" H 6900 2900 60  0000 C CNN
@@
 P 4800 4950
 F 0 "U?" H 5050 4825 60  0000 L CNN
-F 1 "NE5532" H 5025 4750 60  0000 L CNN
+F 1 "OP275" H 5025 4750 60  0000 L CNN
 F 2 "" H 4800 4950 60  0000 C CNN
 F 3 "" H 4800 4950 60  0000 C CNN
@@
 P 6900 5050
 F 0 "U?" H 6900 5350 60  0000 L CNN
-F 1 "NE5532" H 6900 5250 60  0000 L CNN
+F 1 "OP275" H 6900 5250 60  0000 L CNN
 F 2 "~" H 6900 5050 60  0000 C CNN
 F 3 "~" H 6900 5050 60  0000 C CNN
