File: hardware/design/Main Board/Sheet 4.sch (KiCad schematic (older format))
At the start: 22 parts

Commit message: Added Power Ports
Connections:
- net labels added: VDD, VSS
- wire segments 48 -> 52
Changed lines of the file:
@@
 Sheet 4 5
 Title ""
-Date "17 apr 2014"
+Date "29 apr 2014"
 Rev ""
 Comp ""
@@
 U 1 1 534EAE4C
 P 5700 1750
-F 0 "C?" V 5750 1800 30  0000 L CNN
-F 1 "0.1u" V 5750 1650 30  0000 L CNN
+F 0 "C?" V 5790 1640 30  0000 L CNN
+F 1 "0.1u" V 5750 1630 30  0000 L CNN
 F 2 "~" H 5700 1750 60  0000 C CNN
 F 3 "~" H 5700 1750 60  0000 C CNN
@@
 U 1 1 534EAF34
 P 5700 3000
-F 0 "C?" V 5800 2900 30  0000 L CNN
-F 1 "0.1u" V 5750 2900 30  0000 L CNN
+F 0 "C?" V 5760 3030 30  0000 L CNN
+F 1 "0.1u" V 5670 3030 30  0000 L CNN
 F 2 "~" H 5700 3000 60  0000 C CNN
 F 3 "~" H 5700 3000 60  0000 C CNN
@@
 U 1 1 534EB292
 P 5700 4200
-F 0 "C?" V 5750 4250 30  0000 L CNN
-F 1 "0.1u" V 5750 4100 30  0000 L CNN
+F 0 "C?" V 5750 4100 30  0000 L CNN
+F 1 "0.1u" V 5790 4090 30  0000 L CNN
 F 2 "~" H 5700 4200 60  0000 C CNN
 F 3 "~" H 5700 4200 60  0000 C CNN
@@
 U 1 1 534EB29E
 P 5700 5450
-F 0 "C?" V 5800 5350 30  0000 L CNN
-F 1 "0.1u" V 5750 5350 30  0000 L CNN
+F 0 "C?" V 5770 5470 30  0000 L CNN
+F 1 "0.1u" V 5660 5470 30  0000 L CNN
 F 2 "~" H 5700 5450 60  0000 C CNN
 F 3 "~" H 5700 5450 60  0000 C CNN
@@
 	4750 2350 5050 2350
 Wire Wire Line
-	5600 2800 5600 3000
+	5600 2800 5600 3150
 Wire Wire Line
 	5950 2800 5950 3250
@@
 	6450 3250 6600 3250
 Wire Wire Line
-	5600 1750 5600 1900
+	5600 1650 5600 1900
 Wire Wire Line
 	6250 2350 6600 2350
@@
 	4750 4800 5050 4800
 Wire Wire Line
-	5600 5250 5600 5450
+	5600 5250 5600 5600
 Wire Wire Line
 	5950 5250 5950 5700
@@
 	6450 5700 6600 5700
 Wire Wire Line
-	5600 4200 5600 4350
+	5600 4100 5600 4350
 Wire Wire Line
 	6700 4350 6500 4350
@@
 	5450 4350 5450 4050
 Wire Wire Line
-	6900 2150 6900 2200
+	6900 2100 6900 2200
 Wire Wire Line
 	7100 2150 7100 2250
 Wire Wire Line
-	6900 2750 6900 2700
+	6900 2700 6900 2850
 Wire Wire Line
 	7100 2750 7100 2850
+$Comp
+L VDD #PWR?
+U 1 1 535FB6D3
+P 5600 1650
+F 0 "#PWR?" H 5600 1750 30  0001 C CNN
+F 1 "VDD" H 5600 1760 30  0000 C CNN
+F 2 "" H 5600 1650 60  0000 C CNN
+F 3 "" H 5600 1650 60  0000 C CNN
+	1    5600 1650
+	1    0    0    -1
+$EndComp
+$Comp
+L VDD #PWR?
+U 1 1 535FB6E2
+P 6900 2100
+F 0 "#PWR?" H 6900 2200 30  0001 C CNN
+F 1 "VDD" H 6900 2210 30  0000 C CNN
+F 2 "" H 6900 2100 60  0000 C CNN
+F 3 "" H 6900 2100 60  0000 C CNN
+	1    6900 2100
+	1    0    0    -1
+$EndComp
+$Comp
+L VDD #PWR?
+U 1 1 535FB6F1
+P 6750 2950
+F 0 "#PWR?" H 6750 3050 30  0001 C CNN
+F 1 "VDD" H 6750 3060 30  0000 C CNN
+F 2 "" H 6750 2950 60  0000 C CNN
+F 3 "" H 6750 2950 60  0000 C CNN
+	1    6750 2950
+	1    0    0    -1
+$EndComp
+$Comp
+L VDD #PWR?
+U 1 1 535FB700
+P 5600 4100
+F 0 "#PWR?" H 5600 4200 30  0001 C CNN
+F 1 "VDD" H 5600 4210 30  0000 C CNN
+F 2 "" H 5600 4100 60  0000 C CNN
+F 3 "" H 5600 4100 60  0000 C CNN
+	1    5600 4100
+	1    0    0    -1
+$EndComp
+$Comp
+L VDD #PWR?
+U 1 1 535FB70F
+P 6750 5400
+F 0 "#PWR?" H 6750 5500 30  0001 C CNN
+F 1 "VDD" H 6750 5510 30  0000 C CNN
+F 2 "" H 6750 5400 60  0000 C CNN
+F 3 "" H 6750 5400 60  0000 C CNN
+	1    6750 5400
+	1    0    0    -1
+$EndComp
+$Comp
+L VSS #PWR?
+U 1 1 535FB71E
+P 5600 3150
+F 0 "#PWR?" H 5600 3150 30  0001 C CNN
+F 1 "VSS" H 5600 3080 30  0000 C CNN
+F 2 "" H 5600 3150 60  0000 C CNN
+F 3 "" H 5600 3150 60  0000 C CNN
+	1    5600 3150
+	1    0    0    -1
+$EndComp
+$Comp
+L VSS #PWR?
+U 1 1 535FB72D
+P 5600 5600
+F 0 "#PWR?" H 5600 5600 30  0001 C CNN
+F 1 "VSS" H 5600 5530 30  0000 C CNN
+F 2 "" H 5600 5600 60  0000 C CNN
+F 3 "" H 5600 5600 60  0000 C CNN
+	1    5600 5600
+	1    0    0    -1
+$EndComp
+$Comp
+L VSS #PWR?
+U 1 1 535FB73C
+P 6750 6050
+F 0 "#PWR?" H 6750 6050 30  0001 C CNN
+F 1 "VSS" H 6750 5980 30  0000 C CNN
+F 2 "" H 6750 6050 60  0000 C CNN
+F 3 "" H 6750 6050 60  0000 C CNN
+	1    6750 6050
+	1    0    0    -1
+$EndComp
+$Comp
+L VSS #PWR?
+U 1 1 535FB74B
+P 6750 3600
+F 0 "#PWR?" H 6750 3600 30  0001 C CNN
+F 1 "VSS" H 6750 3530 30  0000 C CNN
+F 2 "" H 6750 3600 60  0000 C CNN
+F 3 "" H 6750 3600 60  0000 C CNN
+	1    6750 3600
+	1    0    0    -1
+$EndComp
+$Comp
+L VSS #PWR?
+U 1 1 535FB75A
+P 6900 2850
+F 0 "#PWR?" H 6900 2850 30  0001 C CNN
+F 1 "VSS" H 6900 2780 30  0000 C CNN
+F 2 "" H 6900 2850 60  0000 C CNN
+F 3 "" H 6900 2850 60  0000 C CNN
+	1    6900 2850
+	1    0    0    -1
+$EndComp
+Connection ~ 5600 1750
+Connection ~ 5600 3000
+Connection ~ 6900 2150
+Connection ~ 6900 2750
+Wire Wire Line
+	6750 3000 6750 2950
+Wire Wire Line
+	6750 3500 6750 3600
+Connection ~ 5600 4200
+Connection ~ 5600 5450
+Wire Wire Line
+	6750 5450 6750 5400
+Wire Wire Line
+	6750 5950 6750 6050
 $EndSCHEMATC
