File: hardware/design/Main Board/Sheet 5.sch (KiCad schematic (older format))
At the start: 26 parts

Commit message: Added Power Ports
Connections:
- net labels added: VDD, VSS
- wire segments 66 -> 74
Changed lines of the file:
@@
 Sheet 5 5
 Title ""
-Date "17 apr 2014"
+Date "29 apr 2014"
 Rev ""
 Comp ""
@@
 Text HLabel 7350 4800 2    60   Output ~ 0
 CH2-_OUT
+$Comp
+L VSS #PWR?
+U 1 1 535FBDF9
+P 3700 3150
+F 0 "#PWR?" H 3700 3150 30  0001 C CNN
+F 1 "VSS" H 3700 3080 30  0000 C CNN
+F 2 "" H 3700 3150 60  0000 C CNN
+F 3 "" H 3700 3150 60  0000 C CNN
+	1    3700 3150
+	1    0    0    -1
+$EndComp
+$Comp
+L VSS #PWR?
+U 1 1 535FBE08
+P 3700 5150
+F 0 "#PWR?" H 3700 5150 30  0001 C CNN
+F 1 "VSS" H 3700 5080 30  0000 C CNN
+F 2 "" H 3700 5150 60  0000 C CNN
+F 3 "" H 3700 5150 60  0000 C CNN
+	1    3700 5150
+	1    0    0    -1
+$EndComp
+$Comp
+L VSS #PWR?
+U 1 1 535FBE17
+P 5500 3150
+F 0 "#PWR?" H 5500 3150 30  0001 C CNN
+F 1 "VSS" H 5500 3080 30  0000 C CNN
+F 2 "" H 5500 3150 60  0000 C CNN
+F 3 "" H 5500 3150 60  0000 C CNN
+	1    5500 3150
+	1    0    0    -1
+$EndComp
+$Comp
+L VDD #PWR?
+U 1 1 535FBE35
+P 3700 4050
+F 0 "#PWR?" H 3700 4150 30  0001 C CNN
+F 1 "VDD" H 3700 4160 30  0000 C CNN
+F 2 "" H 3700 4050 60  0000 C CNN
+F 3 "" H 3700 4050 60  0000 C CNN
+	1    3700 4050
+	1    0    0    -1
+$EndComp
+$Comp
+L VDD #PWR?
+U 1 1 535FBE44
+P 4900 4050
+F 0 "#PWR?" H 4900 4150 30  0001 C CNN
+F 1 "VDD" H 4900 4160 30  0000 C CNN
+F 2 "" H 4900 4050 60  0000 C CNN
+F 3 "" H 4900 4050 60  0000 C CNN
+	1    4900 4050
+	1    0    0    -1
+$EndComp
+$Comp
+L VDD #PWR?
+U 1 1 535FBE53
+P 3700 2050
+F 0 "#PWR?" H 3700 2150 30  0001 C CNN
+F 1 "VDD" H 3700 2160 30  0000 C CNN
+F 2 "" H 3700 2050 60  0000 C CNN
+F 3 "" H 3700 2050 60  0000 C CNN
+	1    3700 2050
+	1    0    0    -1
+$EndComp
+$Comp
+L VDD #PWR?
+U 1 1 535FBE62
+P 4900 2000
+F 0 "#PWR?" H 4900 2100 30  0001 C CNN
+F 1 "VDD" H 4900 2110 30  0000 C CNN
+F 2 "" H 4900 2000 60  0000 C CNN
+F 3 "" H 4900 2000 60  0000 C CNN
+	1    4900 2000
+	1    0    0    -1
+$EndComp
+Wire Wire Line
+	4900 2100 4900 2000
+Connection ~ 4900 2100
+Wire Wire Line
+	3700 2050 3700 2100
+Wire Wire Line
+	3700 3100 3700 3150
+Wire Wire Line
+	3700 4050 3700 4100
+Wire Wire Line
+	3700 5100 3700 5150
+Wire Wire Line
+	4900 4050 4900 4100
+Connection ~ 4900 4100
+$Comp
+L VSS #PWR?
+U 1 1 535FC0CC
+P 5500 5150
+F 0 "#PWR?" H 5500 5150 30  0001 C CNN
+F 1 "VSS" H 5500 5080 30  0000 C CNN
+F 2 "" H 5500 5150 60  0000 C CNN
+F 3 "" H 5500 5150 60  0000 C CNN
+	1    5500 5150
+	1    0    0    -1
+$EndComp
+Wire Wire Line
+	5500 5100 5500 5150
+Connection ~ 5500 5100
+Wire Wire Line
+	5500 3100 5500 3150
+Connection ~ 5500 3100
 $EndSCHEMATC
