File: hardware/design/Main Board/Sheet 6.sch (KiCad schematic (older format))
At the start: 24 parts

Commit message: Version 1.0.082514.2134
Initial partial PCB layout.
Parts:
- added P23, P24, P25, P26: TST, ~, symbol TST
- gave numbers to parts that had none: 22
Connections:
- wire segments 66 -> 68

Commit message: Version 1.0.090114.2238
Completed Layout
Parts:
- added R104, R105: 0, ~, symbol R
Connections:
- wire segments 68 -> 70
Changed lines of the file:
@@
 Sheet 6 9
 Title "Hybrid Audio Dynamics Processor"
-Date "26 aug 2014"
+Date "2 sep 2014"
 Rev "1.0"
 Comp "P14345"
@@
 Text HLabel 1750 4800 0    60   Input ~ 0
 LPF_IN_2
-Text HLabel 7600 3100 2    60   Output ~ 0
+Text HLabel 8200 3100 2    60   Output ~ 0
 LPF_OUT_1
-Text HLabel 7600 5000 2    60   Output ~ 0
+Text HLabel 8200 5000 2    60   Output ~ 0
 LPF_OUT_2
 $Comp
@@
 	7500 4950 7500 5000
 Connection ~ 7500 5000
+$Comp
+L R R104
+U 1 1 54052E3B
+P 7850 3100
+F 0 "R104" V 7930 3100 40  0000 C CNN
+F 1 "0" V 7857 3101 40  0000 C CNN
+F 2 "~" V 7780 3100 30  0000 C CNN
+F 3 "~" H 7850 3100 30  0000 C CNN
+	1    7850 3100
+	0    -1   -1   0
+$EndComp
+$Comp
+L R R105
+U 1 1 54052E4A
+P 7850 5000
+F 0 "R105" V 7930 5000 40  0000 C CNN
+F 1 "0" V 7857 5001 40  0000 C CNN
+F 2 "~" V 7780 5000 30  0000 C CNN
+F 3 "~" H 7850 5000 30  0000 C CNN
+	1    7850 5000
+	0    -1   -1   0
+$EndComp
+Wire Wire Line
+	8100 3100 8200 3100
+Wire Wire Line
+	8100 5000 8200 5000
 $EndSCHEMATC
