File: hardware/design/Main Board/Sheet 7.sch (KiCad schematic (older format))
At the start: 15 parts

Commit message: Version 1.0
Wrapped up design. Version for Detailed Design Review.
Parts:
- removed P?: CONN_17, symbol CONN_17
- removed RV?: 10K, ~, symbol POT
- added C? (x2): 1u, ~, symbol CP1
- added C? (x2): 100n, ~, symbol C
- added C? (x2): 100n, ~, symbol CSMALL
- added P?: ROT_ENC, symbol CONN_4
- added P?: DISP, symbol CONN_2
- added R? (x2): 6.2K, ~, symbol R
- added R? (x12): 10K, ~, symbol R
Connections:
- net labels added: CH1_CV, CH1_MUG, CH2_CV, CH2_MUG, RELAY_1, RELAY_2, VDDA, VREF+
- net labels removed: +5V, D0, D1, D2, D3, D4, D5, D6, D7, E, RS, RW
- wire segments 90 -> 192
- no-connect marks 1 -> 4
Other:
- moved on the sheet: C?, K?

Commit message: Version 1.0.05112014.1736
Updated Sheet Sizes
Added Voltage Divider
Parts:
- added R? (x2): 22K, ~, symbol R
- added R? (x2): 1K, ~, symbol R
Connections:
- wire segments 192 -> 200
Other:
- moved on the sheet: C?, K?, P?, R?, SW?, U?, X?

Commit message: Version 1.0.051414.2106
- Added JTAG & Programming Port to MCU.
- Moved I2C Display to the I2C2 Buss.
- Added 10K reference resistors.
Parts:
- added P?: JTAG, symbol CONN_10X2
- added P?: PROG, symbol CONN_2
- added R? (x3): 10K, ~, symbol R
Connections:
- net labels added: JNTRST, JTCK, JTDI, JTDO, JTSM, NRST
- wire segments 200 -> 235
- no-connect marks 4 -> 3
Other:
- moved on the sheet: C?, K?, P?, R?, SW?, U?, X?

Commit message: Version 1.0.082514.2134
Initial partial PCB layout.
Parts:
- removed R? (x2): 10K, ~, symbol R
- added R38, R57: 10K, ~, symbol R
- added R41, R43, R44, R55: 0, ~, symbol R
- added RP1, RP3, RP6, RP7, RP8, RP9: 0 Ohm, ~, symbol R_PACK8
- added RP2, RP4, RP5: 0 Ohm, ~, symbol R_PACK4
- gave numbers to parts that had none: 42
Connections:
- net labels added: OSC_IN, OSC_OUT
- wire segments 235 -> 334
- no-connect marks 3 -> 1
Other:
- moved on the sheet: C49, C50, P27, P28, P30, R37, R39, R40, R42, R45, R50, R52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
