File: hardware/design/Main Board/Sheet 1.kicad_pcb (KiCad board)
At the start: 4 copper layers, 126.5 x 61.6 mm, 211 parts, among them K1 CONN_3, K2 PANASONIC_TX-S, K3 PANASONIC_TX-S, P1 CONN_4, P10 TST, P11 TST, P12 TST, P13 TST, P14 TST, P15 TST, P16 TST, P17 TST, P18 TST, P19 TST, P2 CONN_4, P20 TST, P21 TST, P22 TST, P23 TST, P24 TST, P25 TST, P26 TST, P27 PROG, P28 ROT_ENC, P29 JTAG, P3 TST, P30 DISP, P4 TST, P40 CONN_2, P41 CONN_2, P5 TST, P6 TST, P7 TST, P8 TST, P9 TST, Q1 BSS138, Q2 BSS138, Q5 MMBF170, Q6 MMBF170, SW1 SW_PUSH, U1 OP275, U10 OP275, U11 STM32F303XC, U2 OP275, U3 OP275, U4 THAT2181, U5 THAT2181, U6 OP275, U7 THAT1646, U8 THAT1646, U9 OP275, X1 24MHz

Commit message: Version 1.0.090114.2238
Completed Layout
Parts:
- added P100: TST, PINTST, F.Cu at (120.3, 144.6)
- added P101: TST, PINTST, F.Cu at (52.7, 158.0)
- added P102: TST, PINTST, F.Cu at (54.0, 137.0)
- added P103: TST, PINTST, F.Cu at (44.8, 111.5)
- added P104: TST, PINTST, F.Cu at (72.1, 115.9)
- added P105: TST, PINTST, F.Cu at (62.7, 150.4)
- added P106: TST, PINTST, F.Cu at (126.4, 148.4)
- added P107: TST, PINTST, F.Cu at (114.8, 114.8)
- added P108: TST, PINTST, F.Cu at (119.0, 112.0)
- added P109: TST, PINTST, F.Cu at (26.0, 108.9)
- added P110: TST, PINTST, F.Cu at (40.9, 110.7)
- added P111: TST, PINTST, F.Cu at (70.9, 158.8)
- added P200: CONN_5, PIN_ARRAY_5x1, F.Cu at (20.4, 111.4)
- added R100: 0, SM0603_Resistor, B.Cu at (40.0, 134.4)
- added R101: 0, SM0603_Resistor, B.Cu at (40.8, 136.2)
- added R102: 0, SM0603_Resistor, F.Cu at (71.9, 127.5)
- added R103: 0, SM0603_Resistor, F.Cu at (66.2, 144.7)
- added R104: 0, SM0603_Resistor, F.Cu at (47.2, 111.2)
- added R105: 0, SM0603_Resistor, F.Cu at (43.0, 151.9)
- added R106: 0, SM0603_Resistor, F.Cu at (62.5, 125.5)
- added R107: 0, SM0603_Resistor, F.Cu at (60.0, 147.6)
- added R108: 0, SM0603_Resistor, F.Cu at (50.1, 131.4)
- added R109: 0, SM0603_Resistor, F.Cu at (52.6, 131.4)
- added R110: 0, SM0603_Resistor, F.Cu at (50.9, 138.7)
- added R111: 0, SM0603_Resistor, F.Cu at (49.1, 144.2)
- added R112: 0, SM0603_Resistor, F.Cu at (84.9, 121.4)
- added R113: 0, SM0603_Resistor, F.Cu at (85.1, 111.0)
- added R114: R, SM0603_Resistor, F.Cu at (85.3, 160.7)
- added R115: R, SM0603_Resistor, F.Cu at (84.2, 149.8)
- moved P26 3.66 mm to (43.6, 150.0)
- moved P18 1.34 mm to (64.0, 145.6)
Connections:
- C21 pad 2: /Output Stage/CH1_LN_DVR_IN -> N-0000066
- C22 pad 2: /Output Stage/CH2_LN_DVR_IN -> N-0000062
- C33 pad 1: /Output Stage/CH1-_OUT -> N-0000076
- C34 pad 1: /Output Stage/CH2-_OUT -> N-0000075
- C35 pad 1: /Output Stage/CH1+_OUT -> N-0000077
- C36 pad 1: /Output Stage/CH2+_OUT -> N-0000074
- C47 pad 2: /Precision Rectifier/CH1_RECT_IN -> N-0000096
- C48 pad 2: /Precision Rectifier/CH2_RECT_IN -> N-0000089
- C7 pad 1: /Input Section/CH1 -> N-0000039
- C8 pad 1: /Input Section/CH2 -> N-0000031
- FB1 pad 2: /Output Stage/CH1+_OUT -> N-0000077
- FB2 pad 2: /Output Stage/CH1-_OUT -> N-0000076
- FB3 pad 2: /Output Stage/CH2+_OUT -> N-0000074
- FB4 pad 2: /Output Stage/CH2-_OUT -> N-0000075
- P11 pad 1: /MCU/A_IN_1 -> N-0000047
- P12 pad 1: /MCU/A_IN_2 -> N-0000044
- P15 pad 1: /Output Stage/CH1_LN_DVR_IN -> N-0000066
- P16 pad 1: /Output Stage/CH2_LN_DVR_IN -> N-0000062
- P19 pad 1: /Output Stage/CH1+_OUT -> N-0000077
- P20 pad 1: /Output Stage/CH1-_OUT -> N-0000076
- P21 pad 1: /Output Stage/CH2+_OUT -> N-0000074
- P22 pad 1: /Output Stage/CH2-_OUT -> N-0000075
- P25 pad 1: /Precision Rectifier/CH1_RECT_IN -> N-0000096
- P26 pad 1: /Precision Rectifier/CH2_RECT_IN -> N-0000089
- P7 pad 1: /Input Section/CH1 -> N-0000039
- P8 pad 1: /Input Section/CH2 -> N-0000031
- R11 pad 1: /Input Section/CH1 -> N-0000039
- R12 pad 1: /Input Section/CH2 -> N-0000031
- R21 pad 2: /MCU/A_IN_1 -> N-0000047
- R22 pad 2: /MCU/A_IN_2 -> N-0000044
- R27 pad 2: /Output Stage/CH1_LN_DVR_IN -> N-0000066
- R28 pad 2: /Output Stage/CH2_LN_DVR_IN -> N-0000062
- U1 pad 1: /Input Section/CH1 -> N-0000039
- U1 pad 7: /Input Section/CH2 -> N-0000031
- U10 pad 6: /Precision Rectifier/CH2_RECT_IN -> N-0000089
- U10 pad 7: /Precision Rectifier/CH2_RECT_IN -> N-0000089
- U2 pad 7: /MCU/A_IN_1 -> N-0000047
- U3 pad 7: /MCU/A_IN_2 -> N-0000044
- U4 pad 2: /VCA Section/CH1_CV+ -> N-0000053
- U4 pad 3: /MCU/CH1_CV -> N-0000054
- U5 pad 2: /VCA Section/CH2_CV+ -> N-0000056
- U5 pad 3: /MCU/CH2_CV -> N-0000055
- U6 pad 1: /Output Stage/CH1_LN_DVR_IN -> N-0000066
- U6 pad 7: /Output Stage/CH2_LN_DVR_IN -> N-0000062
- U9 pad 5: /Precision Rectifier/CH1_RECT_IN -> N-0000096
- U9 pad 7: /Precision Rectifier/CH1_RECT_IN -> N-0000096
Routing:
- net VDD: track 19.2 -> 291.9 mm, vias 0 -> 13
- net VSS: track 20.9 -> 230.2 mm, vias 0 -> 10
- net +5V: track 0.00 -> 139.0 mm
- net +3.3V: track 158.5 -> 260.9 mm
- net N-0000089: track 0.00 -> 14.6 mm
- net /MCU/A_IN_1: track 77.9 -> 63.4 mm
- net N-0000096: track 0.00 -> 14.0 mm
- net N-0000047: track 0.00 -> 13.1 mm
- net /Output Stage/CH2_LN_DVR_IN: track 16.1 -> 3.99 mm
- net /Precision Rectifier/CH2_RECT_IN: track 17.1 -> 5.14 mm
- net N-0000062: track 0.00 -> 11.9 mm
- net N-0000044: track 0.00 -> 11.1 mm
- net N-0000039: track 0.00 -> 10.8 mm, vias 0 -> 1
- net /MCU/A_IN_2: track 63.4 -> 53.1 mm
- net /Output Stage/CH2+_OUT: track 18.2 -> 8.34 mm
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Other:
- net class VDD added: clearance 0.508, trace_width 0.508, via_dia 0.508, via_drill 0.3302
- net class VSS added: clearance 0.508, trace_width 0.508, via_dia 0.508, via_drill 0.3302

Commit message: Version 1.0.090814.2105
Gerbers
Parts:
- removed P10, P13, P14, P23, P24, P9: TST, PINTST
- added M3-HOLE: VAL**, M3-HOLE, F.Cu at (156.8, 161.9)
- added M3-HOLE: VAL**, M3-HOLE, F.Cu at (274.3, 109.2)
- added M3-HOLE: VAL**, M3-HOLE, F.Cu at (274.3, 161.9)
- added M3-HOLE: VAL**, M3-HOLE, F.Cu at (169.5, 118.7)
- moved P2 137.9 mm to (274.9, 136.7)
- moved C1 137.9 mm to (166.3, 134.0)
- moved C10 137.9 mm to (173.9, 135.8)
- moved C11 137.9 mm to (198.8, 125.1)
- moved C12 137.9 mm to (195.9, 114.2)
- moved C13 137.9 mm to (201.0, 159.6)
- moved C14 137.9 mm to (195.1, 150.9)
- moved C15 137.9 mm to (183.6, 136.1)
- moved C16 137.9 mm to (183.6, 139.1)
- moved C17 137.9 mm to (198.3, 133.8)
- moved C18 137.9 mm to (194.7, 133.8)
- moved C19 137.9 mm to (198.3, 141.4)
- moved C2 137.9 mm to (166.3, 126.4)
- moved C20 137.9 mm to (194.7, 141.4)
- moved C21 137.9 mm to (207.4, 132.5)
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